File: onestacker_butbetter.kicad_pcb (KiCad board)
At the start: 2 copper layers, 104 parts, among them J1 Conn_01x05, J10 Conn_01x01, J11 Conn_01x01, J12 Conn_01x01, J2 Conn_01x02, J3 Conn_01x02, J4 Conn_01x03, J5 Conn_01x03, J6 Conn_01x03, J7 Conn_01x03, J8 Conn_01x13, J9 Conn_01x01, Q1 BSS138, Q10 BSS138, Q11 BSS138, Q12 BSS138, Q13 NSV1C201MZ4, Q2 BSS138, Q3 BSS138, Q4 BSS138, Q5 BSS138, Q6 BSS138, Q7 BSS138, Q8 BSS138, Q9 BSS138, T1 HX1188NL, U1 LTC6804-1

Commit message: fixed package issue
Parts:
- U1: footprint 6804-1:6804-1-LTC6804-1 -> SOP50P780X200-48N:SOP50P780X200-48N
- moved U1 1.45 mm to (128.5, 93.0)
Routing:
- net Net-(R4-Pad1): track 0.00 -> 27.6 mm
- net Net-(R6-Pad1): track 0.00 -> 25.5 mm
- net Net-(R46-Pad1): track 0.00 -> 25.4 mm
- net Net-(R44-Pad1): track 0.00 -> 24.1 mm
- net Net-(R8-Pad1): track 0.00 -> 23.7 mm
- net Net-(R42-Pad1): track 0.00 -> 23.2 mm
- net Net-(R10-Pad1): track 0.00 -> 22.3 mm
- net Net-(R40-Pad1): track 0.00 -> 21.8 mm
- net Net-(R12-Pad1): track 0.00 -> 20.0 mm
- net Net-(R14-Pad1): track 0.00 -> 18.2 mm
- net Net-(R38-Pad1): track 0.00 -> 18.0 mm
- net Net-(R16-Pad1): track 0.00 -> 16.5 mm
- net Net-(R18-Pad1): track 0.00 -> 15.6 mm
- net Net-(R36-Pad1): track 0.90 -> 16.0 mm
- net Net-(R20-Pad1): track 0.00 -> 14.7 mm
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